File: serial-port-upgrade.sch (KiCad schematic (older format))
At the start: 10 parts, among them J1 MFP 7 RC, J2 MFP 11 VCC, J3 MFP 16 TDO, J4 MFP 18 XTAL2, J5 MFP 34 /IEI, J6 MFP 36 GND, SW1 MOD ENABLE, U1 4040

Commit message: added some notes about my additions to the mod
Other:
- note added: "I added an optionnal bypass capacitor."
- note added: "The original mod takes into account that \npin 34 of the MFP is tied to ground on \nthe ST. I added an optionnal way to use \nthe real GND pin of the MFP."
Changed lines of the file:
@@
 NoConn ~ 4450 5500
 NoConn ~ 4450 5600
+Text Notes 2850 6100 2    50   ~ 0
+The original mod takes into account that \npin 34 of the MFP is tied to ground on \nthe ST. I added an optionnal way to use \nthe real GND pin of the MFP.
+Text Notes 3050 4100 2    50   ~ 0
+I added an optionnal bypass capacitor.
 $EndSCHEMATC

Commit message: PCB done
Parts:
- C1: footprint (none) -> commons-passives_THT:Passive_THT_capacitor_W2.54mm_L10.16mm
- J1, J2, J3, J4, J5, J6: footprint (none) -> Connector_PinHeader_2.54mm:PinHeader_1x01_P2.54mm_Vertical
- JP1: footprint (none) -> Jumper:SolderJumper-3_P1.3mm_Bridged12_RoundedPad1.0x1.5mm
- SW1: footprint (none) -> Connector_PinHeader_2.54mm:PinHeader_1x03_P2.54mm_Horizontal
- U1: footprint (none) -> Package_DIP:DIP-16_W7.62mm_Socket_LongPads
Connections:
- net at U1.7 (Q1): now also SW1.1 (A); no longer SW1.3 (C)
- net at J3.1 (Pin_1): now also SW1.3 (C); no longer SW1.1 (A)
Changed lines of the file:
@@
 F 0 "U1" H 3650 5650 50  0000 C CNN
 F 1 "4040" H 3650 4250 50  0000 C CNN
-F 2 "" H 3950 5000 50  0001 C CNN
+F 2 "Package_DIP:DIP-16_W7.62mm_Socket_LongPads" H 3950 5000 50  0001 C CNN
 F 3 "http://www.intersil.com/content/dam/Intersil/documents/cd40/cd4020bms-24bms-40bms.pdf" H 3950 5000 50  0001 C CNN
 	1    3950 5000
@@
 F 0 "J1" H 2450 3100 50  0000 C CNN
 F 1 "MFP 7 RC" H 2450 2900 50  0000 C CNN
-F 2 "" H 2450 3000 50  0001 C CNN
+F 2 "Connector_PinHeader_2.54mm:PinHeader_1x01_P2.54mm_Vertical" H 2450 3000 50  0001 C CNN
 F 3 "~" H 2450 3000 50  0001 C CNN
 	1    2450 3000
@@
 F 0 "J2" H 2450 3900 50  0000 C CNN
 F 1 "MFP 11 VCC" H 2450 3700 50  0000 C CNN
-F 2 "" H 2450 3800 50  0001 C CNN
+F 2 "Connector_PinHeader_2.54mm:PinHeader_1x01_P2.54mm_Vertical" H 2450 3800 50  0001 C CNN
 F 3 "~" H 2450 3800 50  0001 C CNN
 	1    2450 3800
@@
 F 0 "J4" H 2450 4600 50  0000 C CNN
 F 1 "MFP 18 XTAL2" H 2450 4400 50  0000 C CNN
-F 2 "" H 2450 4500 50  0001 C CNN
+F 2 "Connector_PinHeader_2.54mm:PinHeader_1x01_P2.54mm_Vertical" H 2450 4500 50  0001 C CNN
 F 3 "~" H 2450 4500 50  0001 C CNN
 	1    2450 4500
@@
 F 0 "J5" H 2450 4900 50  0000 C CNN
 F 1 "MFP 34 /IEI" H 2450 4700 50  0000 C CNN
-F 2 "" H 2450 4800 50  0001 C CNN
+F 2 "Connector_PinHeader_2.54mm:PinHeader_1x01_P2.54mm_Vertical" H 2450 4800 50  0001 C CNN
 F 3 "~" H 2450 4800 50  0001 C CNN
 	1    2450 4800
@@
 F 0 "J6" H 2450 5600 50  0000 C CNN
 F 1 "MFP 36 GND" H 2450 5400 50  0000 C CNN
-F 2 "" H 2450 5500 50  0001 C CNN
+F 2 "Connector_PinHeader_2.54mm:PinHeader_1x01_P2.54mm_Vertical" H 2450 5500 50  0001 C CNN
 F 3 "~" H 2450 5500 50  0001 C CNN
 	1    2450 5500
@@
 F 0 "J3" H 5650 3000 50  0000 C CNN
 F 1 "MFP 16 TDO" H 5650 2800 50  0000 C CNN
-F 2 "" H 5650 2900 50  0001 C CNN
+F 2 "Connector_PinHeader_2.54mm:PinHeader_1x01_P2.54mm_Vertical" H 5650 2900 50  0001 C CNN
 F 3 "~" H 5650 2900 50  0001 C CNN
 	1    5650 2900
@@
 F 0 "SW1" H 3900 3170 50  0000 C CNN
 F 1 "MOD ENABLE" H 3900 2800 50  0000 C CNN
-F 2 "" H 3900 3000 50  0001 C CNN
+F 2 "Connector_PinHeader_2.54mm:PinHeader_1x03_P2.54mm_Horizontal" H 3900 3000 50  0001 C CNN
 F 3 "~" H 3900 3000 50  0001 C CNN
 	1    3900 3000
-	1    0    0    -1
+	1    0    0    1
 $EndComp
 $Comp
@@
 F 0 "JP1" H 2850 5400 50  0000 C CNN
 F 1 "GND source" H 2950 5610 50  0000 C CNN
-F 2 "" H 2950 5500 50  0001 C CNN
+F 2 "Jumper:SolderJumper-3_P1.3mm_Bridged12_RoundedPad1.0x1.5mm" H 2950 5500 50  0001 C CNN
 F 3 "~" H 2950 5500 50  0001 C CNN
 	1    2950 5500
@@
 F 0 "C1" H 3300 4150 50  0000 L CNN
 F 1 "0.1uF" H 3300 3950 50  0000 L CNN
-F 2 "" H 3250 4050 50  0001 C CNN
+F 2 "commons-passives_THT:Passive_THT_capacitor_W2.54mm_L10.16mm" H 3250 4050 50  0001 C CNN
 F 3 "~" H 3250 4050 50  0001 C CNN
 	1    3250 4050
