File: serial-port-upgrade.kicad_pcb (KiCad board)
At the start: 2 copper layers, 19 x 46.7 mm, 12 parts, among them J1 MFP 7 RC, J2 MFP 11 VCC, J3 MFP 16 TDO, J4 MFP 18 XTAL2, J5 MFP 34 /IEI, J6 MFP 36 GND, SW1 MOD ENABLE, U1 4040

Commit message: added some annotation
Routing:
- net /mod_gnd: vias 6 -> 3
- net (no net): vias 0 -> 3
Other:
- board text added: "MFP 1"
Changed lines of the file:
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@@
   (general
     (thickness 1.6)
-    (drawings 18)
+    (drawings 20)
     (tracks 47)
     (zones 0)
@@
       (net 2 "Net-(C1-Pad1)"))
   )
+  (gr_text "MFP 1" (at 76.2 104.902 90) (layer F.SilkS)
+    (effects (font (size 1 1) (thickness 0.15)))
+  )
+  (gr_poly (pts (xy 76.962 102.362) (xy 75.438 102.362) (xy 75.438 100.838) (xy 76.962 100.838)) (layer F.SilkS) (width 0.1))
   (gr_text https://github.com (at 76.327 100.457 90) (layer B.SilkS)
     (effects (font (size 1 1) (thickness 0.15)) (justify left mirror))
@@
   (via (at 90.297 134.62) (size 0.762) (drill 0.381) (layers F.Cu B.Cu) (net 1))
   (via (at 85.598 130.302) (size 0.762) (drill 0.381) (layers F.Cu B.Cu) (net 1))
-  (via (at 76.2 134.62) (size 0.762) (drill 0.381) (layers F.Cu B.Cu) (net 1))
-  (via (at 76.581 142.24) (size 0.762) (drill 0.381) (layers F.Cu B.Cu) (net 1))
-  (via (at 91.567 142.621) (size 0.762) (drill 0.381) (layers F.Cu B.Cu) (net 1))
+  (via (at 76.2 134.62) (size 0.762) (drill 0.381) (layers F.Cu B.Cu) (net 0))
+  (via (at 76.581 142.24) (size 0.762) (drill 0.381) (layers F.Cu B.Cu) (net 0))
+  (via (at 91.567 142.621) (size 0.762) (drill 0.381) (layers F.Cu B.Cu) (net 0))
   (via (at 81.661 132.08) (size 0.762) (drill 0.381) (layers F.Cu B.Cu) (net 1))
   (segment (start 88.9 108.966) (end 88.519 109.347) (width 0.508) (layer F.Cu) (net 2))
